File: doc/schemat/steam_clk/steam_clk.kicad_pcb (KiCad board)
At the start: 2 copper layers, 53.8 x 35.1 mm, 24 parts, among them J1 Goldpin, J2 Cell+, J3 Cell-, SW1 POWER, SW2 SET, SW3 CLEAR, U1 BQ-M322RD, U2 STM32F030F4Px, U3 TC1185-3.3VCT8, Y1 18.432MHz

Commit message: added name on PCB
Other:
- board text added: "CHRONOMETR"
Changed lines of the file:
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@@
   (general
     (thickness 1.6)
-    (drawings 6)
+    (drawings 7)
     (tracks 222)
     (zones 0)
@@
       (rotate (xyz 0 0 0))
     )
+  )
+  (gr_text CHRONOMETR (at 249.428 149.606) (layer F.Cu)
+    (effects (font (size 1.5 1.5) (thickness 0.3)))
   )
   (gr_line (start 258.572 157.48) (end 258.572 122.428) (layer Edge.Cuts) (width 0.1))
@@
     (polygon
       (pts
-        (xy 258.572 122.428) (xy 258.572 157.48) (xy 204.724 157.48) (xy 204.724 122.428)
+        (xy 258.572 122.447995) (xy 258.572 157.499995) (xy 204.724 157.499995) (xy 204.724 122.447995)
       )
     )
