File: doc/project/steam_clk/steam_clk.sch (KiCad schematic (older format))
At the start: 24 parts, among them J1 Goldpin, J2 Cell+, J3 Cell-, SW1 POWER, SW2 SET, SW3 CLEAR, U1 BQ-M322RD, U2 STM32F030F4Px, U3 TC1185-3.3VCT8, Y1 18.432MHz

Commit message: better tracks on pcb
Parts:
- SW2, SW3: footprint Button_Switch_SMD:SW_SPST_B3U-1000P -> Button_Switch_THT:SW_PUSH_6mm_H13mm
Changed lines of the file:
@@
 F 0 "SW2" H 5550 4300 50  0000 C CNN
 F 1 "SET" H 5600 4200 50  0000 C CNN
-F 2 "Button_Switch_SMD:SW_SPST_B3U-1000P" H 5500 4300 50  0001 C CNN
+F 2 "Button_Switch_THT:SW_PUSH_6mm_H13mm" H 5500 4300 50  0001 C CNN
 F 3 "~" H 5500 4300 50  0001 C CNN
 	1    5500 4100
@@
 F 0 "SW3" H 5450 4300 50  0000 C CNN
 F 1 "CLEAR" H 5450 4200 50  0000 C CNN
-F 2 "Button_Switch_SMD:SW_SPST_B3U-1000P" H 5500 4600 50  0001 C CNN
+F 2 "Button_Switch_THT:SW_PUSH_6mm_H13mm" H 5500 4600 50  0001 C CNN
 F 3 "~" H 5500 4600 50  0001 C CNN
 	1    5500 4400
