File: doc/project/daily_clk/daily_clk.sch (KiCad schematic (older format))
At the start: 24 parts, among them J1 Goldpin, J2 Cell+, J3 Cell-, SW1 POWER, SW2 SET, SW3 CLEAR, U1 BQ-M322RD, U2 STM32F030F4Px, U3 TC1185-3.3VCT8, Y1 18.432MHz

Commit message: dodana wersja daily, uaktualnione footprinty przycisków
Parts:
- removed C5: 100u, Capacitor_THT:CP_Radial_D5.0mm_P2.50mm, symbol Device:C
Changed lines of the file:
@@
 EESchema Schematic File Version 4
-LIBS:steam_clk-cache
+LIBS:daily_clk-cache
 EELAYER 29 0
 EELAYER END
@@
 Wire Wire Line
 	5400 5700 4800 5700
-Wire Wire Line
-	1750 2700 3250 2700
 $Comp
 L power:+3V3 #PWR02
@@
 	5400 5300 5650 5300
 Connection ~ 5400 5300
-Wire Wire Line
-	1750 4700 2200 4700
-Wire Wire Line
-	1750 3550 1750 4700
-Wire Wire Line
-	1750 3250 1750 2700
 Connection ~ 4050 4700
 Connection ~ 5700 4400
@@
 	1    0    0    -1
 $EndComp
-$Comp
-L Device:C C5
-U 1 1 5D1D34FD
-P 1750 3400
-F 0 "C5" H 1865 3446 50  0000 L CNN
-F 1 "100u" H 1865 3355 50  0000 L CNN
-F 2 "Capacitor_THT:CP_Radial_D5.0mm_P2.50mm" H 1788 3250 50  0001 C CNN
-F 3 "~" H 1750 3400 50  0001 C CNN
-	1    1750 3400
-	1    0    0    -1
-$EndComp
