File: doc/project/daily_clk/daily_clk.kicad_pcb (KiCad board)
At the start: 2 copper layers, 66.5 x 59.9 mm, 23 parts, among them J1 Goldpin, J2 Cell+, J3 Cell-, SW1 POWER, SW2 SET, SW3 CLEAR, U1 BQ-M322RD, U2 STM32F030F4Px, U3 TC1185-3.3VCT8, Y1 18.432MHz

Commit message: atomic board
Parts:
- moved C2 26.8 mm to (210.3, 115.3)
- moved C1 24.8 mm to (215.1, 115.3)
- moved U2 23.9 mm to (228.6, 110.7), turned to 0 degrees
- moved C3 13.8 mm to (237.2, 104.1), turned to 270 degrees
- moved U3 9.67 mm to (241.0, 105.7)
- moved R9 7.94 mm to (205.7, 105.4), turned to 270 degrees
- moved SW1 7.15 mm to (222.0, 116.8)
- moved SW3 7.15 mm to (214.3, 119.6), turned to 180 degrees
- moved SW2 7.15 mm to (208.9, 119.6)
- moved J1 7.08 mm to (241.3, 119.4)
- moved J3 6.93 mm to (240.3, 114.8)
- moved J2 6.93 mm to (244.6, 114.8)
- moved C4 6.65 mm to (244.3, 106.7)
- moved R8 6.37 mm to (205.7, 108.7), turned to 270 degrees
- moved Y1 6.14 mm to (210.3, 112.8)
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Routing:
- net SE: track 0.00 -> 59.5 mm, vias 0 -> 2
- net D1: track 0.00 -> 53.2 mm, vias 0 -> 2
- net SF: track 0.00 -> 47.9 mm, vias 0 -> 2
- net +3V3: track 0.00 -> 45.6 mm, vias 0 -> 2
- net Net-(SW2-Pad1): track 0.00 -> 41.5 mm, vias 0 -> 3
- net GND: track 0.00 -> 37.2 mm, vias 0 -> 3
- net Net-(C3-Pad1): track 0.00 -> 36.8 mm, vias 0 -> 2
- net D3: track 0.00 -> 35.4 mm, vias 0 -> 1
- net Net-(R8-Pad1): track 0.00 -> 25.2 mm, vias 0 -> 2
- net D2: track 0.00 -> 24.0 mm, vias 0 -> 2
- net Net-(R9-Pad2): track 0.00 -> 22.2 mm
- net SA: track 0.00 -> 21.6 mm
- net Net-(SW3-Pad1): track 0.00 -> 19.8 mm, vias 0 -> 1
- net Net-(C2-Pad1): track 0.00 -> 19.5 mm
- net Net-(J3-Pad1): track 0.00 -> 18.7 mm
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- added copper zone on B.Cu, net GND
- added copper zone on F.Cu, net GND
Other:
- board size 66.5 x 59.9 mm -> 45.2 x 30.2 mm
