File: doc/project/atomic_clk/atomic_clk.kicad_pcb.kicad_pcb (KiCad board)
At the start: 2 copper layers, 45.2 x 30.2 mm, 23 parts, among them J1 Goldpin, J2 Cell+, J3 Cell-, SW1 POWER, SW2 SET, SW3 CLEAR, U1 BQ-M322RD, U2 STM32F030F4Px, U3 TC1185-3.3VCT8, Y1 18.432MHz

Commit message: atomic update
Parts:
- moved J1 2.29 mm to (239.0, 119.4)
- moved Y1 0.51 mm to (210.8, 112.8)
Routing:
- net GND: track 37.2 -> 30.9 mm
- net Net-(C3-Pad1): track 36.8 -> 38.4 mm
- net D1: track 53.2 -> 54.2 mm
- added copper zone on B.Cu, net (none)
- added copper zone on F.Cu, net (none)
Other:
- board size 45.2 x 30.2 mm -> 47.8 x 30.2 mm
- board text added: "ATOMIC"
- board text added: "by Bart"
