File: doc/project/atomic_clk/atomic_clk.sch (KiCad schematic (older format))
At the start: 23 parts, among them J1 Goldpin, J2 Cell+, J3 Cell-, SW1 POWER, SW2 SET, SW3 CLEAR, U1 BQ-M322RD, U2 STM32F030F4Px, U3 TC1185-3.3VCT8, Y1 18.432MHz

Commit message: przygotowanie pod nowy akumulator
Parts:
- SW2, SW3: footprint Button_Switch_SMD:SW_SPST_CK_KXT3 -> Button_Switch_SMD:SW_SPST_CK_RS282G05A3
Changed lines of the file:
@@
 EESchema Schematic File Version 4
-LIBS:daily_clk-cache
+LIBS:atomic_clk-cache
 EELAYER 29 0
 EELAYER END
@@
 F 0 "SW2" H 5550 4300 50  0000 C CNN
 F 1 "SET" H 5600 4200 50  0000 C CNN
-F 2 "Button_Switch_SMD:SW_SPST_CK_KXT3" H 5500 4300 50  0001 C CNN
+F 2 "Button_Switch_SMD:SW_SPST_CK_RS282G05A3" H 5500 4300 50  0001 C CNN
 F 3 "~" H 5500 4300 50  0001 C CNN
 	1    5500 4100
@@
 F 0 "SW3" H 5450 4300 50  0000 C CNN
 F 1 "CLEAR" H 5450 4200 50  0000 C CNN
-F 2 "Button_Switch_SMD:SW_SPST_CK_KXT3" H 5500 4600 50  0001 C CNN
+F 2 "Button_Switch_SMD:SW_SPST_CK_RS282G05A3" H 5500 4600 50  0001 C CNN
 F 3 "~" H 5500 4600 50  0001 C CNN
 	1    5500 4400

Commit message: jst conetor
Parts:
- removed J2: Cell+, Connector_PinHeader_2.54mm:PinHeader_1x01_P2.54mm_Vertical, symbol Connector:Conn_01x01_Female
- removed J3: Cell-, Connector_PinHeader_2.54mm:PinHeader_1x01_P2.54mm_Vertical, symbol Connector:Conn_01x01_Female
- added J2: Bat, Connector_PinHeader_1.27mm:PinHeader_1x02_P1.27mm_Vertical, symbol Connector:Conn_01x02_Female
Connections:
- net at SW1.2 (B): now also J2.1 (Pin_1)
- net at C3.1, J1.1 (Pin_1), U3.1 (Vin)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: now also J2.2 (Pin_2)
Changed lines of the file:
@@
 Wire Wire Line
 	3200 5700 3900 5700
-$Comp
-L Connector:Conn_01x01_Female J2
-U 1 1 5D1EF089
-P 2150 5300
-F 0 "J2" H 2042 5075 50  0000 C CNN
-F 1 "Cell+" H 2042 5166 50  0000 C CNN
-F 2 "Connector_PinHeader_2.54mm:PinHeader_1x01_P2.54mm_Vertical" H 2150 5300 50  0001 C CNN
-F 3 "~" H 2150 5300 50  0001 C CNN
-	1    2150 5300
-	-1   0    0    1
-$EndComp
-$Comp
-L Connector:Conn_01x01_Female J3
-U 1 1 5D1EFE3D
-P 2150 5600
-F 0 "J3" H 2042 5375 50  0000 C CNN
-F 1 "Cell-" H 2042 5466 50  0000 C CNN
-F 2 "Connector_PinHeader_2.54mm:PinHeader_1x01_P2.54mm_Vertical" H 2150 5600 50  0001 C CNN
-F 3 "~" H 2150 5600 50  0001 C CNN
-	1    2150 5600
-	-1   0    0    1
-$EndComp
 Wire Wire Line
 	2350 5300 3200 5300
@@
 Text Label 3900 700  0    50   ~ 0
 Display
+$Comp
+L Connector:Conn_01x02_Female J2
+U 1 1 5D2E3615
+P 2150 5400
+F 0 "J2" H 2050 5100 50  0000 C CNN
+F 1 "Bat" H 2042 5166 50  0000 C CNN
+F 2 "Connector_PinHeader_1.27mm:PinHeader_1x02_P1.27mm_Vertical" H 2150 5400 50  0001 C CNN
+F 3 "~" H 2150 5400 50  0001 C CNN
+	1    2150 5400
+	-1   0    0    1
+$EndComp
+Wire Wire Line
+	2350 5600 2350 5400
 $EndSCHEMATC
